Commit message: Added V0.2 CAD models and updated URDF

File: flat_bot_support/urdf/flat_bot_macro.xacro (robot description, xacro)
@@ -5,14 +5,14 @@
     <link name="${prefix}sirom_a_link">
       <visual>
-        <origin xyz="0 0 0" rpy="0 0 0"/>
+        <origin xyz="0 0 0" rpy="${-pi/2.0} 0 0"/>
         <geometry>
-          <mesh filename="package://flat_bot_support/meshes/visual/test.dae"/>
+          <mesh filename="package://flat_bot_support/meshes/visual/Sirom_Link.stl" scale="0.001 0.001 0.001"/>
         </geometry>
         <!--xacro:material_fanuc_gray40 /-->
       </visual>
       <collision>
-        <origin xyz="0 0 0" rpy="0 0 0"/>
+        <origin xyz="0 0 0" rpy="${-pi/2.0} 0 0"/>
         <geometry>
-          <mesh filename="package://flat_bot_support/meshes/visual/test.dae"/>
+          <mesh filename="package://flat_bot_support/meshes/visual/Sirom_Link.stl" scale="0.001 0.001 0.001"/>
         </geometry>
       </collision>
@@ -20,14 +20,14 @@
     <link name="${prefix}link_a">
       <visual>
-        <origin xyz="0 0 0" rpy="0 0 0"/>
+        <origin xyz="-0.0785 0.0213 0" rpy="${-pi/2.0} 0 0"/>
         <geometry>
-          <mesh filename="package://flat_bot_support/meshes/visual/test_1.dae"/>
+          <mesh filename="package://flat_bot_support/meshes/visual/Link_A.stl" scale="0.001 0.001 0.001"/>
         </geometry>
         <!--xacro:material_fanuc_gray40 /-->
       </visual>
       <collision>
-        <origin xyz="0 0 0" rpy="0 0 0"/>
+        <origin xyz="-0.0785 0.0213 0" rpy="${-pi/2.0} 0 0"/>
         <geometry>
-          <mesh filename="package://flat_bot_support/meshes/visual/test_1.dae"/>
+          <mesh filename="package://flat_bot_support/meshes/visual/Link_A.stl" scale="0.001 0.001 0.001"/>
         </geometry>
       </collision>
@@ -35,14 +35,14 @@
     <link name="${prefix}link_b">
       <visual>
-        <origin xyz="0 0 0" rpy="0 0 0"/>
+        <origin xyz="${-0.0785 - 0.25} 0.0213 0" rpy="${-pi/2.0} 0 0"/>
         <geometry>
-          <mesh filename="package://flat_bot_support/meshes/visual/test_2.dae"/>
+          <mesh filename="package://flat_bot_support/meshes/visual/Link_B.stl" scale="0.001 0.001 0.001"/>
         </geometry>
         <!--xacro:material_fanuc_gray40 /-->
       </visual>
       <collision>
-        <origin xyz="0 0 0" rpy="0 0 0"/>
+        <origin xyz="${-0.0785 - 0.25} 0.0213 0" rpy="${-pi/2.0} 0 0"/>
         <geometry>
-          <mesh filename="package://flat_bot_support/meshes/visual/test_2.dae"/>
+          <mesh filename="package://flat_bot_support/meshes/visual/Link_B.stl" scale="0.001 0.001 0.001"/>
         </geometry>
       </collision>
@@ -50,14 +50,14 @@
     <link name="${prefix}sirom_b_link">
       <visual>
-        <origin xyz="0 0 0" rpy="0 0 0"/>
+        <origin xyz="0.0785 -0.0213 0" rpy="${-pi/2.0} 0 ${pi}"/>
         <geometry>
-          <mesh filename="package://flat_bot_support/meshes/visual/test_3.dae"/>
+          <mesh filename="package://flat_bot_support/meshes/visual/Sirom_Link_2.stl" scale="0.001 0.001 0.001"/>
         </geometry>
         <!--xacro:material_fanuc_gray40 /-->
       </visual>
       <collision>
-        <origin xyz="0 0 0" rpy="0 0 0"/>
+        <origin xyz="0.0785 -0.021 0" rpy="${-pi/2.0} 0 ${pi}"/>
         <geometry>
-          <mesh filename="package://flat_bot_support/meshes/visual/test_3.dae"/>
+          <mesh filename="package://flat_bot_support/meshes/visual/Sirom_Link_2.stl" scale="0.001 0.001 0.001"/>
         </geometry>
       </collision>
@@ -65,5 +65,5 @@
     <!-- joints: main serial chain -->
     <joint name="${prefix}wrist_a_joint" type="revolute">
-      <origin xyz="0 0 0" rpy="0 0 0"/>
+      <origin xyz="0.0785 -0.0213 0" rpy="0 0 0"/>
       <parent link="${prefix}sirom_a_link"/>
       <child link="${prefix}link_a"/>
@@ -72,5 +72,5 @@
     </joint>
     <joint name="${prefix}elbow_joint" type="revolute">
-      <origin xyz="2 0 0" rpy="0 0 0"/>
+      <origin xyz="0.25 0 0" rpy="0 0 0"/>
       <parent link="${prefix}link_a"/>
       <child link="${prefix}link_b"/>
@@ -79,5 +79,5 @@
     </joint>
     <joint name="${prefix}wrist_b_joint" type="revolute">
-      <origin xyz="2 0 0" rpy="0 0 0"/>
+      <origin xyz="0.25 0 0" rpy="0 0 0"/>
       <parent link="${prefix}link_b"/>
       <child link="${prefix}sirom_b_link"/>

Commit message: Corrected Sirom frames in Flatbot URDF file

File: flat_bot_support/urdf/flat_bot_macro.xacro (robot description, xacro)
@@ -88,5 +88,5 @@
     <link name="${prefix}sirom_a_origin" />
     <joint name="${prefix}sirom_a_origin-link" type="fixed">
-      <origin xyz="0.5 0 0" rpy="0 0 0"/>
+      <origin xyz="0 0 0" rpy="0 0 ${pi}"/>
       <parent link="${prefix}sirom_a_origin"/>
       <child link="${prefix}sirom_a_link"/>
@@ -95,5 +95,5 @@
     <link name="${prefix}sirom_b_origin" />
     <joint name="${prefix}sirom_b_link-origin" type="fixed">
-      <origin xyz="0.5 0 0" rpy="0 0 ${pi}" />
+      <origin xyz="0.0785 -0.0213 0" rpy="0 0 0" />
       <parent link="${prefix}sirom_b_link" />
       <child link="${prefix}sirom_b_origin" />

Commit message: Converted flatbot models to collada

File: flat_bot_support/urdf/flat_bot_macro.xacro (robot description, xacro)
@@ -7,5 +7,5 @@
         <origin xyz="0 0 0" rpy="${-pi/2.0} 0 0"/>
         <geometry>
-          <mesh filename="package://flat_bot_support/meshes/visual/Sirom_Link.stl" scale="0.001 0.001 0.001"/>
+          <mesh filename="package://flat_bot_support/meshes/visual/Sirom_Link.dae" scale="0.001 0.001 0.001"/>
         </geometry>
         <!--xacro:material_fanuc_gray40 /-->
@@ -14,5 +14,5 @@
         <origin xyz="0 0 0" rpy="${-pi/2.0} 0 0"/>
         <geometry>
-          <mesh filename="package://flat_bot_support/meshes/visual/Sirom_Link.stl" scale="0.001 0.001 0.001"/>
+          <mesh filename="package://flat_bot_support/meshes/visual/Sirom_Link.dae" scale="0.001 0.001 0.001"/>
         </geometry>
       </collision>
@@ -22,5 +22,5 @@
         <origin xyz="-0.0785 0.0213 0" rpy="${-pi/2.0} 0 0"/>
         <geometry>
-          <mesh filename="package://flat_bot_support/meshes/visual/Link_A.stl" scale="0.001 0.001 0.001"/>
+          <mesh filename="package://flat_bot_support/meshes/visual/Link_A.dae" scale="0.001 0.001 0.001"/>
         </geometry>
         <!--xacro:material_fanuc_gray40 /-->
@@ -29,5 +29,5 @@
         <origin xyz="-0.0785 0.0213 0" rpy="${-pi/2.0} 0 0"/>
         <geometry>
-          <mesh filename="package://flat_bot_support/meshes/visual/Link_A.stl" scale="0.001 0.001 0.001"/>
+          <mesh filename="package://flat_bot_support/meshes/visual/Link_A.dae" scale="0.001 0.001 0.001"/>
         </geometry>
       </collision>
@@ -37,5 +37,5 @@
         <origin xyz="${-0.0785 - 0.25} 0.0213 0" rpy="${-pi/2.0} 0 0"/>
         <geometry>
-          <mesh filename="package://flat_bot_support/meshes/visual/Link_B.stl" scale="0.001 0.001 0.001"/>
+          <mesh filename="package://flat_bot_support/meshes/visual/Link_B.dae" scale="0.001 0.001 0.001"/>
         </geometry>
         <!--xacro:material_fanuc_gray40 /-->
@@ -44,5 +44,5 @@
         <origin xyz="${-0.0785 - 0.25} 0.0213 0" rpy="${-pi/2.0} 0 0"/>
         <geometry>
-          <mesh filename="package://flat_bot_support/meshes/visual/Link_B.stl" scale="0.001 0.001 0.001"/>
+          <mesh filename="package://flat_bot_support/meshes/visual/Link_B.dae" scale="0.001 0.001 0.001"/>
         </geometry>
       </collision>
@@ -52,5 +52,5 @@
         <origin xyz="0.0785 -0.0213 0" rpy="${-pi/2.0} 0 ${pi}"/>
         <geometry>
-          <mesh filename="package://flat_bot_support/meshes/visual/Sirom_Link_2.stl" scale="0.001 0.001 0.001"/>
+          <mesh filename="package://flat_bot_support/meshes/visual/Sirom_Link_2.dae" scale="0.001 0.001 0.001"/>
         </geometry>
         <!--xacro:material_fanuc_gray40 /-->
@@ -59,5 +59,5 @@
         <origin xyz="0.0785 -0.021 0" rpy="${-pi/2.0} 0 ${pi}"/>
         <geometry>
-          <mesh filename="package://flat_bot_support/meshes/visual/Sirom_Link_2.stl" scale="0.001 0.001 0.001"/>
+          <mesh filename="package://flat_bot_support/meshes/visual/Sirom_Link_2.dae" scale="0.001 0.001 0.001"/>
         </geometry>
       </collision>

Commit message: Got a working Gazebo-MoveIt setup working for the arm!

File: flat_bot_support/urdf/flat_bot_macro.xacro (robot description, xacro)
@@ -2,4 +2,15 @@
 <robot xmlns:xacro="http://wiki.ros.org/xacro">
   <xacro:macro name="flat_bot" params="prefix">
+    <!-- ROS Control Plugin used to drive joints -->
+    <gazebo>
+      <plugin name="gazebo_ros_control" filename="libgazebo_ros_control.so">
+        <!--robotNamespace></robotNamespace-->
+      </plugin>
+    </gazebo>
+    <!-- placeholder links to define the connector coordinate frames of each end effector -->
+    <link name="${prefix}sirom_a_origin">
+    </link>
+    <link name="${prefix}sirom_b_origin">
+    </link>
     <!-- links: main serial chain -->
     <link name="${prefix}sirom_a_link">
@@ -17,4 +28,12 @@
         </geometry>
       </collision>
+    <inertial>
+      <mass value="0.145" />
+      <origin xyz="0.0 0.0 -0.001687" rpy="0.0 0.0 0.0" />
+      <inertia
+	  ixx="0.000065748" ixy="0.0" ixz="0.0"
+	  iyy="0.000065207" iyz="0.0"
+	  izz="0.000058981" />
+    </inertial>
     </link>
     <link name="${prefix}link_a">
@@ -22,5 +41,5 @@
         <origin xyz="-0.0785 0.0213 0" rpy="${-pi/2.0} 0 0"/>
         <geometry>
-          <mesh filename="package://flat_bot_support/meshes/visual/Link_A.dae" scale="0.001 0.001 0.001"/>
+          <mesh filename="package://flat_bot_support/meshes/visual/Link_A.stl" scale="0.001 0.001 0.001"/>
         </geometry>
         <!--xacro:material_fanuc_gray40 /-->
@@ -29,7 +48,15 @@
         <origin xyz="-0.0785 0.0213 0" rpy="${-pi/2.0} 0 0"/>
         <geometry>
-          <mesh filename="package://flat_bot_support/meshes/visual/Link_A.dae" scale="0.001 0.001 0.001"/>
+          <mesh filename="package://flat_bot_support/meshes/visual/Link_A.stl" scale="0.001 0.001 0.001"/>
         </geometry>
       </collision>
+    <inertial>
+      <mass value="0.145" />
+      <origin xyz="0.0 0.0 -0.001687" rpy="0.0 0.0 0.0" />
+      <inertia
+	  ixx="0.000065748" ixy="0.0" ixz="0.0"
+	  iyy="0.000065207" iyz="0.0"
+	  izz="0.000058981" />
+    </inertial>
     </link>
     <link name="${prefix}link_b">
@@ -37,5 +64,5 @@
         <origin xyz="${-0.0785 - 0.25} 0.0213 0" rpy="${-pi/2.0} 0 0"/>
         <geometry>
-          <mesh filename="package://flat_bot_support/meshes/visual/Link_B.dae" scale="0.001 0.001 0.001"/>
+          <mesh filename="package://flat_bot_support/meshes/visual/Link_B.stl" scale="0.001 0.001 0.001"/>
         </geometry>
         <!--xacro:material_fanuc_gray40 /-->
@@ -44,7 +71,15 @@
         <origin xyz="${-0.0785 - 0.25} 0.0213 0" rpy="${-pi/2.0} 0 0"/>
         <geometry>
-          <mesh filename="package://flat_bot_support/meshes/visual/Link_B.dae" scale="0.001 0.001 0.001"/>
+          <mesh filename="package://flat_bot_support/meshes/visual/Link_B.stl" scale="0.001 0.001 0.001"/>
         </geometry>
       </collision>
+    <inertial>
+      <mass value="0.145" />
+      <origin xyz="0.0 0.0 -0.001687" rpy="0.0 0.0 0.0" />
+      <inertia
+	  ixx="0.000065748" ixy="0.0" ixz="0.0"
+	  iyy="0.000065207" iyz="0.0"
+	  izz="0.000058981" />
+    </inertial>
     </link>
     <link name="${prefix}sirom_b_link">
@@ -52,5 +87,5 @@
         <origin xyz="0.0785 -0.0213 0" rpy="${-pi/2.0} 0 ${pi}"/>
         <geometry>
-          <mesh filename="package://flat_bot_support/meshes/visual/Sirom_Link_2.dae" scale="0.001 0.001 0.001"/>
+          <mesh filename="package://flat_bot_support/meshes/visual/Sirom_Link_2.stl" scale="0.001 0.001 0.001"/>
         </geometry>
         <!--xacro:material_fanuc_gray40 /-->
@@ -59,8 +94,22 @@
         <origin xyz="0.0785 -0.021 0" rpy="${-pi/2.0} 0 ${pi}"/>
         <geometry>
-          <mesh filename="package://flat_bot_support/meshes/visual/Sirom_Link_2.dae" scale="0.001 0.001 0.001"/>
+          <mesh filename="package://flat_bot_support/meshes/visual/Sirom_Link_2.stl" scale="0.001 0.001 0.001"/>
         </geometry>
       </collision>
+    <inertial>
+      <mass value="0.145" />
+      <origin xyz="0.0 0.0 -0.001687" rpy="0.0 0.0 0.0" />
+      <inertia
+	  ixx="0.000065748" ixy="0.0" ixz="0.0"
+	  iyy="0.000065207" iyz="0.0"
+	  izz="0.000058981" />
+    </inertial>
     </link>
+    <!-- transforms from the standard SIROM frame to the sirom_a link -->
+    <joint name="${prefix}sirom_a_origin-link" type="fixed">
+      <origin xyz="0 0 0" rpy="0 0 ${pi}"/>
+      <parent link="${prefix}sirom_a_origin"/>
+      <child link="${prefix}sirom_a_link"/>
+    </joint>
     <!-- joints: main serial chain -->
     <joint name="${prefix}wrist_a_joint" type="revolute">
@@ -85,13 +134,5 @@
       <limit lower="${-pi/2.0}" upper="${pi/2.0}" effort="0" velocity="3.67"/>
     </joint>
-    <!-- transforms from the standard SIROM frame to the sirom_a link -->
-    <link name="${prefix}sirom_a_origin" />
-    <joint name="${prefix}sirom_a_origin-link" type="fixed">
-      <origin xyz="0 0 0" rpy="0 0 ${pi}"/>
-      <parent link="${prefix}sirom_a_origin"/>
-      <child link="${prefix}sirom_a_link"/>
-    </joint>
     <!-- transform from the standard SIROM frame to the sirom_b link -->
-    <link name="${prefix}sirom_b_origin" />
     <joint name="${prefix}sirom_b_link-origin" type="fixed">
       <origin xyz="0.0785 -0.0213 0" rpy="0 0 0" />
@@ -99,4 +140,31 @@
       <child link="${prefix}sirom_b_origin" />
     </joint>
+    <transmission name="wrist_a_trans">
+      <type>transmission_interface/SimpleTransmission</type>
+      <joint name="wrist_a_joint">
+        <hardwareInterface>hardware_interface/PositionJointInterface</hardwareInterface>
+      </joint>
+      <actuator name="wrist_a_motor">
+        <mechanicalReduction>50</mechanicalReduction>
+      </actuator>
+    </transmission>
+    <transmission name="elbow_trans">
+      <type>transmission_interface/SimpleTransmission</type>
+      <joint name="elbow_joint">
+        <hardwareInterface>hardware_interface/PositionJointInterface</hardwareInterface>
+      </joint>
+      <actuator name="elbow_motor">
+        <mechanicalReduction>50</mechanicalReduction>
+      </actuator>
+    </transmission>
+    <transmission name="wrist_b_trans">
+      <type>transmission_interface/SimpleTransmission</type>
+      <joint name="wrist_b_joint">
+        <hardwareInterface>hardware_interface/PositionJointInterface</hardwareInterface>
+      </joint>
+      <actuator name="wrist_b_motor">
+        <mechanicalReduction>50</mechanicalReduction>
+      </actuator>
+    </transmission>
   </xacro:macro>
 </robot>

Commit message: tidied up gazebo moveit launch files

File: flat_bot_support/urdf/flat_bot_macro.xacro (robot description, xacro)
@@ -20,5 +20,4 @@
           <mesh filename="package://flat_bot_support/meshes/visual/Sirom_Link.dae" scale="0.001 0.001 0.001"/>
         </geometry>
-        <!--xacro:material_fanuc_gray40 /-->
       </visual>
       <collision>
@@ -29,10 +28,11 @@
       </collision>
     <inertial>
-      <mass value="0.145" />
-      <origin xyz="0.0 0.0 -0.001687" rpy="0.0 0.0 0.0" />
+      <mass value="0.132" />
+      <origin xyz="0.028596 0.0106 -0.023016"
+              rpy="-0.0937241808 0.1033234917 0.1027998929" />
       <inertia
-	  ixx="0.000065748" ixy="0.0" ixz="0.0"
-	  iyy="0.000065207" iyz="0.0"
-	  izz="0.000058981" />
+	  ixx="0.000170585" ixy="0.0" ixz="0.0"
+	  iyy="0.00029451" iyz="0.0"
+	  izz="0.000199521" />
     </inertial>
     </link>
@@ -41,12 +41,11 @@
         <origin xyz="-0.0785 0.0213 0" rpy="${-pi/2.0} 0 0"/>
         <geometry>
-          <mesh filename="package://flat_bot_support/meshes/visual/Link_A.stl" scale="0.001 0.001 0.001"/>
+          <mesh filename="package://flat_bot_support/meshes/visual/Link_A.dae" scale="0.001 0.001 0.001"/>
         </geometry>
-        <!--xacro:material_fanuc_gray40 /-->
       </visual>
       <collision>
-        <origin xyz="-0.0785 0.0213 0" rpy="${-pi/2.0} 0 0"/>
+        <origin xyz="0.250 0 -0.024" rpy="0.0 0.0 0.0" />
         <geometry>
-          <mesh filename="package://flat_bot_support/meshes/visual/Link_A.stl" scale="0.001 0.001 0.001"/>
+          <cylinder length="0.05" radius="0.025" />
         </geometry>
       </collision>
@@ -64,12 +63,11 @@
         <origin xyz="${-0.0785 - 0.25} 0.0213 0" rpy="${-pi/2.0} 0 0"/>
         <geometry>
-          <mesh filename="package://flat_bot_support/meshes/visual/Link_B.stl" scale="0.001 0.001 0.001"/>
+          <mesh filename="package://flat_bot_support/meshes/visual/Link_B.dae" scale="0.001 0.001 0.001"/>
         </geometry>
-        <!--xacro:material_fanuc_gray40 /-->
       </visual>
       <collision>
         <origin xyz="${-0.0785 - 0.25} 0.0213 0" rpy="${-pi/2.0} 0 0"/>
         <geometry>
-          <mesh filename="package://flat_bot_support/meshes/visual/Link_B.stl" scale="0.001 0.001 0.001"/>
+          <mesh filename="package://flat_bot_support/meshes/visual/Link_B.dae" scale="0.001 0.001 0.001"/>
         </geometry>
       </collision>
@@ -87,5 +85,5 @@
         <origin xyz="0.0785 -0.0213 0" rpy="${-pi/2.0} 0 ${pi}"/>
         <geometry>
-          <mesh filename="package://flat_bot_support/meshes/visual/Sirom_Link_2.stl" scale="0.001 0.001 0.001"/>
+          <mesh filename="package://flat_bot_support/meshes/visual/Sirom_Link_2.dae" scale="0.001 0.001 0.001"/>
         </geometry>
         <!--xacro:material_fanuc_gray40 /-->
@@ -94,5 +92,5 @@
         <origin xyz="0.0785 -0.021 0" rpy="${-pi/2.0} 0 ${pi}"/>
         <geometry>
-          <mesh filename="package://flat_bot_support/meshes/visual/Sirom_Link_2.stl" scale="0.001 0.001 0.001"/>
+          <mesh filename="package://flat_bot_support/meshes/visual/Sirom_Link_2.dae" scale="0.001 0.001 0.001"/>
         </geometry>
       </collision>

Commit message: fixed floating arm controller bug

File: flat_bot_support/urdf/flat_bot_macro.xacro (robot description, xacro)
@@ -102,4 +102,26 @@
       </inertial>
     </link>
+    <!--link name="${prefix}sirom_b_latch">
+      <visual>
+        <origin xyz="0 0 0" rpy="0 0 0"/>
+        <geometry>
+          <mesh filename="package://flat_bot_support/meshes/visual/sirom_latch_visual.stl" />
+        </geometry>
+      </visual>
+      <collision>
+        <origin xyz="0 0 0" rpy="0 0 0"/>
+        <geometry>
+          <mesh filename="package://flat_bot_support/meshes/collision/sirom_latch_collision.stl" />
+        </geometry>
+      </collision>
+      <inertial>
+        <mass value="0.038" />
+        <origin xyz="-0.021394 -0.001309 0" rpy="0 0 -0.044331363000656" />
+        <inertia
+            ixx="0.000020967" ixy="0.0" ixz="0.0"
+            iyy="0.000007495" iyz="0.0"
+            izz="0.000027196" />
+      </inertial>
+    </link-->
     <!-- transforms from the standard SIROM frame to the sirom_a link -->
     <joint name="${prefix}sirom_a_origin-link" type="fixed">
@@ -114,5 +136,5 @@
       <child link="${prefix}link_a"/>
       <axis xyz="0 0 1"/>
-      <limit lower="${-pi/2.0}" upper="${pi/2.0}" effort="0" velocity="3.67"/>
+      <limit lower="${-pi/2.0}" upper="${pi/2.0}" effort="100" velocity="3.67"/>
     </joint>
     <joint name="${prefix}elbow_joint" type="revolute">
@@ -121,5 +143,5 @@
       <child link="${prefix}link_b"/>
       <axis xyz="0 0 1"/>
-      <limit lower="-2.96706" upper="2.96706" effort="0" velocity="3.32"/>
+      <limit lower="-2.96706" upper="2.96706" effort="100" velocity="3.32"/>
     </joint>
     <joint name="${prefix}wrist_b_joint" type="revolute">
@@ -128,6 +150,13 @@
       <child link="${prefix}sirom_b_link"/>
       <axis xyz="0 0 1"/>
-      <limit lower="${-pi/2.0}" upper="${pi/2.0}" effort="0" velocity="3.67"/>
-    </joint>
+      <limit lower="${-pi/2.0}" upper="${pi/2.0}" effort="100" velocity="3.67"/>
+    </joint>
+    <!--joint name="${prefix}latch_b_joint" type="revolute">
+      <origin xyz="0.0565 -0.021472 0.038" rpy="0 0 ${-pi/4}"/>
+      <parent link="${prefix}sirom_b_link"/>
+      <child link="${prefix}sirom_b_latch"/>
+      <axis xyz="0 0 1"/>
+      <limit lower="${-pi/2.0}" upper="${pi/2.0}" effort="100" velocity="3.67"/>
+    </joint-->
     <!-- transform from the standard SIROM frame to the sirom_b link -->
     <joint name="${prefix}sirom_b_link-origin" type="fixed">
@@ -136,8 +165,9 @@
       <child link="${prefix}sirom_b_origin" />
     </joint>
+    <!-- ================= Arm Joint Transmissions ==================== -->
     <transmission name="wrist_a_trans">
       <type>transmission_interface/SimpleTransmission</type>
-      <joint name="wrist_a_joint">
-        <hardwareInterface>hardware_interface/PositionJointInterface</hardwareInterface>
+      <joint name="${prefix}wrist_a_joint">
+        <hardwareInterface>hardware_interface/EffortJointInterface</hardwareInterface>
       </joint>
       <actuator name="wrist_a_motor">
@@ -147,6 +177,6 @@
     <transmission name="elbow_trans">
       <type>transmission_interface/SimpleTransmission</type>
-      <joint name="elbow_joint">
-        <hardwareInterface>hardware_interface/PositionJointInterface</hardwareInterface>
+      <joint name="${prefix}elbow_joint">
+        <hardwareInterface>hardware_interface/EffortJointInterface</hardwareInterface>
       </joint>
       <actuator name="elbow_motor">
@@ -156,6 +186,6 @@
     <transmission name="wrist_b_trans">
       <type>transmission_interface/SimpleTransmission</type>
-      <joint name="wrist_b_joint">
-        <hardwareInterface>hardware_interface/PositionJointInterface</hardwareInterface>
+      <joint name="${prefix}wrist_b_joint">
+        <hardwareInterface>hardware_interface/EffortJointInterface</hardwareInterface>
       </joint>
       <actuator name="wrist_b_motor">
@@ -163,4 +193,14 @@
       </actuator>
     </transmission>
+    <!-- ================= SIROM Joint Transmissions ==================== -->
+    <!--transmission name="sirom_latch_b_trans">
+      <type>transmission_interface/SimpleTransmission</type>
+      <joint name="${prefix}latch_b_joint">
+        <hardwareInterface>hardware_interface/EffortJointInterface</hardwareInterface>
+      </joint>
+      <actuator name="latch_b_motor">
+        <mechanicalReduction>50</mechanicalReduction>
+      </actuator>
+    </transmission-->
   </xacro:macro>
 </robot>
